Commit message: Add person follower node and update robot simulation
Introduced a new ROS2 node for person following using MediaPipe Pose and depth camera data. Updated robot URDF and xacro files to support ROS2 control in simulation, added depth camera configuration, and included controller YAML file. Modified launch file to start the person follower and controllers, and adjusted Gazebo world and bridge scripts for improved simulation integration.

File: src/sim_env/description/camera_sensor_macro.xacro (robot description, xacro)
@@ -2,5 +2,5 @@
 <robot xmlns:xacro="http://www.ros.org/wiki/xacro">
   <xacro:macro name="camera_sensor_macro">
-    <sensor name="camera_sensor" type="camera">
+    <sensor name="camera_sensor" type="rgbd_camera">
       <update_rate>30</update_rate>
       <always_on>true</always_on>
@@ -14,7 +14,20 @@
         <clip>
           <near>0.01</near>
-          <far>100</far>
+          <far>20.0</far>
         </clip>
       </camera>
+      <!-- Depth camera part -->
+      <depth_camera>
+        <image>
+          <width>800</width>
+          <height>600</height>
+          <!-- typical depth format -->
+          <format>R_FLOAT32</format>
+        </image>
+        <clip>
+          <near>0.01</near>
+          <far>20.0</far>
+        </clip>
+      </depth_camera>
     </sensor>
   </xacro:macro>

File: src/sim_env/description/cbrn_robot.urdf.xacro (robot description, xacro)
@@ -1,11 +1,14 @@
 <?xml version="1.0"?>
 <robot xmlns:xacro="http://www.ros.org/wiki/xacro" name="cbrn_robot">
-  <!-- <xacro:if value="$(arg use_ros2_control)">
+  <xacro:arg name="use_ros2_control" default="true"/>
+  <xacro:arg name="sim_mode" default="false"/>
+  <xacro:include filename="robot_core.xacro" />
+  <xacro:include filename="camera.xacro" />
+  <xacro:if value="$(arg use_ros2_control)">
     <xacro:include filename="ros2_control.xacro" />
+    <xacro:diff_drive_ros2_control sim_mode="$(arg sim_mode)"/>
   </xacro:if>
   <xacro:unless value="$(arg use_ros2_control)">
     <xacro:include filename="gazebo_control.xacro" />
-  </xacro:unless> -->
-  <xacro:include filename="robot_core.xacro" />
-  <xacro:include filename="camera.xacro" />
+  </xacro:unless>
 </robot>

File: src/sim_env/description/robot_core.xacro (robot description, xacro)
@@ -1,5 +1,5 @@
 <?xml version="1.0"?>
 <robot xmlns:xacro="http://www.ros.org/wiki/xacro" >
-    <!-- <xacro:include filename="inertial_macros.xacro"/>
+    <xacro:include filename="inertial_macros.xacro"/>
     <xacro:property name="chassis_length" value="0.335"/>
     <xacro:property name="chassis_width" value="0.265"/>
@@ -15,23 +15,13 @@
     <xacro:property name="caster_wheel_mass" value="0.01"/>
     <xacro:property name="caster_wheel_offset_x" value="0.075"/>
-    <xacro:property name="caster_wheel_offset_z" value="${wheel_offset_z - wheel_radius + caster_wheel_radius}"/> -->
-    <material name="white">
-        <color rgba="1 1 1 1" />
-    </material>
-    <material name="orange">
-        <color rgba="1 0.3 0.1 1"/>
-    </material>
-    <material name="blue">
-        <color rgba="0.2 0.2 1 1"/>
-    </material>
-    <material name="black">
-        <color rgba="0 0 0 1"/>
-    </material>
-    <material name="red">
-        <color rgba="1 0 0 1"/>
-    </material>
+    <xacro:property name="caster_wheel_offset_z" value="${wheel_offset_z - wheel_radius + caster_wheel_radius}"/>
+    <material name="white"><color rgba="1 1 1 1" /></material>
+    <material name="orange"><color rgba="1 0.3 0.1 1"/></material>
+    <material name="blue"><color rgba="0.2 0.2 1 1"/></material>
+    <material name="black"><color rgba="0 0 0 1"/></material>
+    <material name="red"><color rgba="1 0 0 1"/></material>
     <!-- BASE LINK -->
     <link name="base_link">
-        <visual>
+        <!-- <visual>
         <geometry><box size="0.5 0.3 0.1"/></geometry>
         </visual>
@@ -42,8 +32,8 @@
         <mass value="5.0"/>
         <inertia ixx="0.1" ixy="0.0" ixz="0.0" iyy="0.1" iyz="0.0" izz="0.1"/>
-        </inertial>
+        </inertial> -->
     </link>
     <!-- BASE_FOOTPRINT LINK -->
-    <!-- <joint name="base_footprint_joint" type="fixed">
+    <joint name="base_footprint_joint" type="fixed">
         <parent link="base_link"/>
         <child link="base_footprint"/>
@@ -51,7 +41,7 @@
     </joint>
     <link name="base_footprint">
-    </link> -->
+    </link>
     <!-- CHASSIS LINK -->
-    <!-- <joint name="chassis_joint" type="fixed">
+    <joint name="chassis_joint" type="fixed">
         <parent link="base_link"/>
         <child link="chassis"/>
@@ -72,5 +62,5 @@
             </geometry>
         </collision>
-        <xacro:inertial_box mass="0.5" x="${chassis_length}" y="${chassis_width}" z="${chassis_height}">
+        <xacro:inertial_box mass="5.5" x="${chassis_length}" y="${chassis_width}" z="${chassis_height}">
             <origin xyz="${chassis_length/2} 0 ${chassis_height/2}" rpy="0 0 0"/>
         </xacro:inertial_box>
@@ -78,7 +68,7 @@
     <gazebo reference="chassis">
         <material>Gazebo/Orange</material>
-    </gazebo> -->
+    </gazebo>
     <!-- LEFT WHEEL LINK -->
-    <!-- <joint name="left_wheel_joint" type="continuous">
+    <joint name="left_wheel_joint" type="continuous">
         <parent link="base_link"/>
         <child link="left_wheel"/>
@@ -95,5 +85,5 @@
         <collision>
             <geometry>
-                <sphere radius="${wheel_radius}"/>
+                <cylinder radius="${wheel_radius}" length="${wheel_thickness}"/>
             </geometry>
         </collision>
@@ -104,7 +94,9 @@
     <gazebo reference="left_wheel">
         <material>Gazebo/Blue</material>
-    </gazebo> -->
+        <mu1>1.0</mu1>
+        <mu2>1.0</mu2>
+    </gazebo>
     <!-- RIGHT WHEEL LINK -->
-    <!-- <joint name="right_wheel_joint" type="continuous">
+    <joint name="right_wheel_joint" type="continuous">
         <parent link="base_link"/>
         <child link="right_wheel"/>
@@ -121,5 +113,5 @@
         <collision>
             <geometry>
-                <sphere radius="${wheel_radius}"/>
+                <cylinder radius="${wheel_radius}" length="${wheel_thickness}"/>
             </geometry>
         </collision>
@@ -130,7 +122,9 @@
     <gazebo reference="right_wheel">
         <material>Gazebo/Blue</material>
-    </gazebo> -->
+        <mu1>1.0</mu1>
+        <mu2>1.0</mu2>
+    </gazebo>
     <!-- CASTER WHEEL LINK -->
-    <!-- <joint name="caster_wheel_joint" type="fixed">
+    <joint name="caster_wheel_joint" type="fixed">
         <parent link="chassis"/>
         <child link="caster_wheel"/>
@@ -157,4 +151,4 @@
         <mu1 value="0.001"/>
         <mu2 value="0.001"/>
-    </gazebo> -->
+    </gazebo>
 </robot>

File: src/sim_env/description/ros2_control.xacro (robot description, xacro)
@@ -1,62 +1,63 @@
 <?xml version="1.0"?>
 <robot xmlns:xacro="http://www.ros.org/wiki/xacro">
-    <xacro:unless value="$(arg sim_mode)">
-        <ros2_control name="RealRobot" type="system">
-            <hardware>
-                <plugin>diffdrive_arduino/DiffDriveArduino</plugin>
-                <param name="left_wheel_name">left_wheel_joint</param>
-                <param name="right_wheel_name">right_wheel_joint</param>
-                <param name="loop_rate">30</param>
-                <param name="device">/dev/ttyUSB0</param>
-                <param name="baud_rate">57600</param>
-                <param name="timeout">1000</param>
-                <param name="enc_counts_per_rev">3436</param>
-            </hardware>
-            <joint name="left_wheel_joint">
-                <command_interface name="velocity">
-                    <param name="min">-10</param>
-                    <param name="max">10</param>
-                </command_interface>
-                <state_interface name="velocity"/>
-                <state_interface name="position"/>
-            </joint>
-            <joint name="right_wheel_joint">
-                <command_interface name="velocity">
-                    <param name="min">-10</param>
-                    <param name="max">10</param>
-                </command_interface>
-                <state_interface name="velocity"/>
-                <state_interface name="position"/>
-            </joint>
-        </ros2_control>
-    </xacro:unless>
-    <xacro:if value="$(arg sim_mode)">
-        <ros2_control name="GazeboSystem" type="system">
-            <hardware>
-                <plugin>gazebo_ros2_control/GazeboSystem</plugin>
-            </hardware>
-            <joint name="left_wheel_joint">
-                <command_interface name="velocity">
-                    <param name="min">-10</param>
-                    <param name="max">10</param>
-                </command_interface>
-                <state_interface name="velocity"/>
-                <state_interface name="position"/>
-            </joint>
-            <joint name="right_wheel_joint">
-                <command_interface name="velocity">
-                    <param name="min">-10</param>
-                    <param name="max">10</param>
-                </command_interface>
-                <state_interface name="velocity"/>
-                <state_interface name="position"/>
-            </joint>
-        </ros2_control>
-    </xacro:if>
-    <gazebo>
-        <plugin name="gazebo_ros2_control" filename="libgazebo_ros2_control.so">
-            <parameters>$(find articubot_one)/config/my_controllers.yaml</parameters>
-            <parameters>$(find articubot_one)/config/gaz_ros2_ctl_use_sim.yaml</parameters>
-        </plugin>
-    </gazebo>
+    <xacro:macro name="diff_drive_ros2_control" params="sim_mode">
+        <xacro:unless value="${sim_mode}">
+            <ros2_control name="RealRobot" type="system">
+                <hardware>
+                    <plugin>diffdrive_arduino/DiffDriveArduino</plugin>
+                    <param name="left_wheel_name">left_wheel_joint</param>
+                    <param name="right_wheel_name">right_wheel_joint</param>
+                    <param name="loop_rate">30</param>
+                    <param name="device">/dev/ttyUSB0</param>
+                    <param name="baud_rate">57600</param>
+                    <param name="timeout">1000</param>
+                    <param name="enc_counts_per_rev">3436</param>
+                </hardware>
+                <joint name="left_wheel_joint">
+                    <command_interface name="velocity">
+                        <param name="min">-10</param>
+                        <param name="max">10</param>
+                    </command_interface>
+                    <state_interface name="velocity"/>
+                    <state_interface name="position"/>
+                </joint>
+                <joint name="right_wheel_joint">
+                    <command_interface name="velocity">
+                        <param name="min">-10</param>
+                        <param name="max">10</param>
+                    </command_interface>
+                    <state_interface name="velocity"/>
+                    <state_interface name="position"/>
+                </joint>
+            </ros2_control>
+        </xacro:unless>
+        <xacro:if value="${sim_mode}">
+            <ros2_control name="GazeboSystem" type="system">
+                <hardware>
+                    <plugin>gz_ros2_control/GazeboSimSystem</plugin>
+                </hardware>
+                <joint name="left_wheel_joint">
+                    <command_interface name="velocity">
+                        <param name="min">-10</param>
+                        <param name="max">10</param>
+                    </command_interface>
+                    <state_interface name="velocity"/>
+                    <state_interface name="position"/>
+                </joint>
+                <joint name="right_wheel_joint">
+                    <command_interface name="velocity">
+                        <param name="min">-10</param>
+                        <param name="max">10</param>
+                    </command_interface>
+                    <state_interface name="velocity"/>
+                    <state_interface name="position"/>
+                </joint>
+            </ros2_control>
+        </xacro:if>
+        <gazebo>
+            <plugin filename="libgz_ros2_control-system.so" name="gz_ros2_control::GazeboSimROS2ControlPlugin">
+                <parameters>$(find sim_env)/config/my_controllers.yaml</parameters>
+            </plugin>
+        </gazebo>
+    </xacro:macro>
 </robot>
