Commit message: Add YOLO detector and update robot config
Introduced yolo_detector.py for person detection using YOLO and depth images. Updated person_follower.py to disable movement logic. Changed wheel link names and added Gazebo parameters in robot_core.xacro. Enabled stamped velocity in my_controllers.yaml. Delayed RViz launch with TimerAction and improved RViz configuration for better visualization.

File: src/sim_env/description/robot_core.xacro (robot description, xacro)
@@ -72,9 +72,9 @@
     <joint name="left_wheel_joint" type="continuous">
         <parent link="base_link"/>
-        <child link="left_wheel"/>
+        <child link="left_wheel_link"/>
         <origin xyz="0 ${wheel_offset_y} 0" rpy="-${pi/2} 0 0" />
         <axis xyz="0 0 1"/>
     </joint>
-    <link name="left_wheel">
+    <link name="left_wheel_link">
         <visual>
             <geometry>
@@ -92,17 +92,20 @@
         </xacro:inertial_cylinder>
     </link>
-    <gazebo reference="left_wheel">
+    <gazebo reference="left_wheel_link">
         <material>Gazebo/Blue</material>
         <mu1>1.0</mu1>
         <mu2>1.0</mu2>
+        <kp>1000000.0</kp>
+        <kd>100.0</kd>
+        <minDepth>0.001</minDepth>
     </gazebo>
     <!-- RIGHT WHEEL LINK -->
     <joint name="right_wheel_joint" type="continuous">
         <parent link="base_link"/>
-        <child link="right_wheel"/>
+        <child link="right_wheel_link"/>
         <origin xyz="0 ${-wheel_offset_y} 0" rpy="${pi/2} 0 0" />
         <axis xyz="0 0 -1"/>
     </joint>
-    <link name="right_wheel">
+    <link name="right_wheel_link">
         <visual>
             <geometry>
@@ -120,8 +123,11 @@
         </xacro:inertial_cylinder>
     </link>
-    <gazebo reference="right_wheel">
+    <gazebo reference="right_wheel_link">
         <material>Gazebo/Blue</material>
         <mu1>1.0</mu1>
         <mu2>1.0</mu2>
+        <kp>1000000.0</kp>
+        <kd>100.0</kd>
+        <minDepth>0.001</minDepth>
     </gazebo>
     <!-- CASTER WHEEL LINK -->
