Commit message: Adjust camera orientation and person pose in simulation
Updated the camera joint's roll-pitch-yaw in camera.xacro for camera to look slightly up (because before I didn't see the head of the human entity). Changed the person_standing model's pose in cbrn_world.world to stand instead of laying down to test if Media Pipe Pose is correctly identifying the person.

File: src/sim_env/description/camera.xacro (robot description, xacro)
@@ -6,5 +6,5 @@
         <parent link="base_link"/>
         <child link="camera_link"/>
-        <origin xyz="0 0 0.2" rpy="0 0 0"/>
+        <origin xyz="0 0 0.2" rpy="0 -0.2 0"/>
     </joint>
     <!-- Link minim pentru camera -->

Commit message: Replace pose/person nodes with new detectors and controller
Removed pose_estimator_node and person_follower, added new detectors (ResNet50, MediaPipe, MoveNet, YOLO) and a robot_controller node. Updated setup.py entry points and launch file to use new nodes. Improved YOLO detector to support pose estimation and CSV export. Adjusted camera and robot model parameters, added a second person to the simulation world, and updated RViz configuration for new TF frames.

File: src/sim_env/description/camera.xacro (robot description, xacro)
@@ -4,7 +4,8 @@
   <!-- Camera joint: poziționează camera pe robot -->
     <joint name="camera_joint" type="fixed">
-        <parent link="base_link"/>
+        <parent link="chassis"/>
         <child link="camera_link"/>
-        <origin xyz="0 0 0.2" rpy="0 -0.2 0"/>
+        <!-- Calcul pentru camera ca sa stea lipita de sasiu -->
+        <origin xyz="${chassis_length} 0 ${chassis_height + 0.025}" rpy="0 -0.2 0"/>
     </joint>
     <!-- Link minim pentru camera -->

File: src/sim_env/description/robot_core.xacro (robot description, xacro)
@@ -4,5 +4,5 @@
     <xacro:property name="chassis_length" value="0.335"/>
     <xacro:property name="chassis_width" value="0.265"/>
-    <xacro:property name="chassis_height" value="0.138"/>
+    <xacro:property name="chassis_height" value="0.25"/>
     <xacro:property name="chassis_mass" value="1.0"/>
     <xacro:property name="wheel_radius" value="0.033"/>

Commit message: Update camera positioning and dimensions in model files

File: src/sim_env/description/camera.xacro (robot description, xacro)
@@ -7,5 +7,5 @@
         <child link="camera_link"/>
         <!-- Calcul pentru camera ca sa stea lipita de sasiu -->
-        <origin xyz="${chassis_length} 0 ${chassis_height + 0.025}" rpy="0 -0.2 0"/>
+        <origin xyz="${chassis_length} 0 ${chassis_height + 0.3}" rpy="0 -0.2 0"/>
     </joint>
     <!-- Link minim pentru camera -->

Commit message: Automate saving png files of models

File: src/sim_env/description/camera.xacro (robot description, xacro)
@@ -7,5 +7,5 @@
         <child link="camera_link"/>
         <!-- Calcul pentru camera ca sa stea lipita de sasiu -->
-        <origin xyz="${chassis_length} 0 ${chassis_height + 0.3}" rpy="0 -0.2 0"/>
+        <origin xyz="${chassis_length} 0 ${chassis_height + 0.5}" rpy="0 -0.2 0"/>
     </joint>
     <!-- Link minim pentru camera -->
