Commit message: Refactor robot controller to use Twist message, enhance movement logic, and add logging for detected distances; update setup and configuration files for new components.

File: src/sim_env/description/cbrn_robot.urdf.xacro (robot description, xacro)
@@ -2,5 +2,5 @@
 <robot xmlns:xacro="http://www.ros.org/wiki/xacro" name="cbrn_robot">
   <xacro:arg name="use_ros2_control" default="true"/>
-  <xacro:arg name="sim_mode" default="false"/>
+  <xacro:arg name="sim_mode" default="true"/>
   <xacro:include filename="robot_core.xacro" />
   <xacro:include filename="camera.xacro" />

File: src/sim_env/description/gazebo_control.xacro (robot description, xacro)
@@ -1,21 +1,21 @@
-<?xml version="1.0"?>
-<robot xmlns:xacro="http://www.ros.org/wiki/xacro">
-    <gazebo>
-        <plugin name="diff_drive" filename="libgazebo_ros_diff_drive.so">
-            <!-- Wheel Information -->
-            <left_joint>left_wheel_joint</left_joint>
-            <right_joint>right_wheel_joint</right_joint>
-            <wheel_separation>0.297</wheel_separation>
-            <wheel_diameter>0.066</wheel_diameter>
-            <!-- Limits -->
-            <max_wheel_torque>200</max_wheel_torque>
-            <max_wheel_acceleration>10.0</max_wheel_acceleration>
-            <!-- Output -->
-            <odometry_frame>odom</odometry_frame>
-            <robot_base_frame>base_link</robot_base_frame>
-            <publish_odom>true</publish_odom>
-            <publish_odom_tf>true</publish_odom_tf>
-            <publish_wheel_tf>true</publish_wheel_tf>
-        </plugin>
-    </gazebo>
-</robot>
+<ros2_control name="GazeboSimSystem" type="system">
+    <hardware>
+        <plugin>gz_ros2_control/GazeboSimSystem</plugin>
+    </hardware>
+    <joint name="left_wheel_joint">
+        <command_interface name="velocity">
+            <param name="min">-10</param>
+            <param name="max">10</param>
+        </command_interface>
+        <state_interface name="position"/>
+        <state_interface name="velocity"/>
+    </joint>
+    <joint name="right_wheel_joint">
+        <command_interface name="velocity">
+            <param name="min">-10</param>
+            <param name="max">10</param>
+        </command_interface>
+        <state_interface name="position"/>
+        <state_interface name="velocity"/>
+    </joint>
+</ros2_control>

File: src/sim_env/description/ros2_control.xacro (robot description, xacro)
@@ -35,5 +35,5 @@
             <ros2_control name="GazeboSystem" type="system">
                 <hardware>
-                    <plugin>gz_ros2_control/GazeboSimSystem</plugin>
+                    <plugin>gz_ros2_control/GazeboSimROS2ControlPlugin</plugin>
                 </hardware>
                 <joint name="left_wheel_joint">
